Commit message: Adds gripper to environment

File: nLinkUrdfReacher/resources/nlink_3.urdf (robot description, URDF)
Before this commit: robot panda_description, 6 links, 5 joints
Links:
- removed link panda_link8
- added link panda_link4, mass 0.0001; collision sphere radius=0.01; visual sphere radius=0.1
Joints:
- removed joint panda_joint8
- added joint panda_joint4: type fixed, parent panda_link3, child panda_link4, origin xyz=0 0 1.2 rpy=0 0 0, axis 0 0 1
