Commit message: Introduces abstractrobot and modify panda and nLinkReacher accordingly

File: pandaReacher/resources/pandaWithGripper_working.urdf (robot description, URDF)
Before this commit: robot panda, 11 links, 10 joints
Links:
- added link world
Joints:
- added joint panda_joint_world: type fixed, parent world, child panda_link0, origin xyz=0 0 0 rpy=0 0 0
