Commit message: Adds visual link as end-effector for boxer robot.

File: boxerRobot/resources/boxer.urdf (robot description, URDF)
Before this commit: robot albert, 22 links, 21 joints
Links:
- added link ee_link; visual sphere radius=0.0625
Joints:
- added joint ee_joint: type fixed, parent base_link, child ee_link, origin xyz=0.6 0 0 rpy=0 0 0

Commit message: Simplifies boxer robot and removes unecessary rotation. Suggests clipping of vel_int.

File: boxerRobot/resources/boxer.urdf (robot description, URDF)
Before this commit: robot albert, 23 links, 22 joints
Links:
- removed link base_footprint
- removed link extrusion1
- removed link extrusion2
- removed link extrusion3
- removed link extrusion4
- removed link front_laser
- removed link imu_link
- removed link internal_link
- removed link lift_link
- removed link rear_left_sonar_link
- removed link rear_right_sonar_link
- removed link stereo
- removed link stereo_left
- removed link stereo_right
- removed link top_mount
- removed link top_mount_bottom
- link chassis_link: mass 51 -> 250
- link rotacastor_left_link: mass 100 -> 1
- link rotacastor_right_link: mass 100 -> 1
- link wheel_left_link: mass 100 -> 10
- link wheel_right_link: mass 100 -> 10
Joints:
- removed joint base_footprint_joint
- removed joint base_laser_joint
- removed joint extrusion1_joint
- removed joint extrusion2_joint
- removed joint extrusion3_joint
- removed joint extrusion4_joint
- removed joint imu_joint
- removed joint internal_joint
- removed joint lift_joint
- removed joint rear_left_sonar_joint
- removed joint rear_right_sonar_joint
- removed joint stereo_camera_joint
- removed joint stereo_left_joint
- removed joint stereo_right_joint
- removed joint top_mount_bottom_joint
- removed joint top_mount_joint
- joint base_chassis_joint: origin xyz=0.15 0 0 rpy=0 0 1.5708 -> xyz=0 0 0 rpy=0 0 0
- joint ee_joint: origin xyz=0.6 0 0 rpy=0 0 0 -> xyz=0 -0.4 0 rpy=0 0 0
