Commit message: Adds home position to panda and albert. Cleans up the changes in the urdf file of albert

File: albertReacher/resources/albert.urdf (robot description, URDF)
Before this commit: robot albert, 34 links, 33 joints
Joints:
- joint mmrobot_joint4: limit lower=-1.50100 upper=1.500996 effort=87 velocity=2.1750 -> lower=-3.0718 upper=0.0698 effort=87 velocity=2.1750; origin xyz=0.0825 0 0 rpy=1.57079632679 1.57079632679 0 -> xyz=0.0825 0 0 rpy=1.57079632679 0 0
- joint mmrobot_joint6: limit lower=-1.58830 upper=2.1817 effort=12 velocity=2.6100 -> lower=-0.0175 upper=3.7525 effort=12 velocity=2.6100; origin xyz=0 0 0 rpy=1.57079632679 -1.57079632679 0 -> xyz=0 0 0 rpy=1.57079632679 0 0

Commit message: Applies similar changes to albertReacher as previously to boxer.

File: albertReacher/resources/albert.urdf (robot description, URDF)
Before this commit: robot albert, 34 links, 33 joints
Links:
- removed link base_footprint
- removed link front_laser
- removed link imu_link
- removed link rear_left_sonar_link
- removed link rear_right_sonar_link
- removed link stereo
- removed link stereo_left
- removed link stereo_right
- link chassis_link: mass 51 -> 250
- link rotacastor_left_link: mass 100 -> 1
- link rotacastor_right_link: mass 100 -> 1
Joints:
- removed joint base_footprint_joint
- removed joint base_laser_joint
- removed joint imu_joint
- removed joint rear_left_sonar_joint
- removed joint rear_right_sonar_joint
- removed joint stereo_camera_joint
- removed joint stereo_left_joint
- removed joint stereo_right_joint
- joint base_chassis_joint: origin xyz=0.15 0 0 rpy=0 0 1.5708 -> xyz=0.0 0 0 rpy=0 0 0
- joint lift_joint: type prismatic -> fixed
