Commit message: Starting to fix the issue with wheels, currently no caster wheels

File: tiagoReacher/resources/tiago_dual.urdf (robot description, URDF)
Before this commit: robot tiago_dual, 69 links, 68 joints
Links:
- removed link base_footprint
- removed link base_mic_back_left_link
- removed link base_mic_back_right_link
- removed link base_mic_front_left_link
- removed link base_mic_front_right_link
- removed link base_sonar_01_link
- removed link base_sonar_02_link
- removed link base_sonar_03_link
- removed link caster_back_left_1_link
- removed link caster_back_left_2_link
- removed link caster_back_right_1_link
- removed link caster_back_right_2_link
- removed link caster_front_left_1_link
- removed link caster_front_left_2_link
- removed link caster_front_right_1_link
- removed link caster_front_right_2_link
- removed link rgbd_laser_link
- removed link xtion_depth_frame
- removed link xtion_depth_optical_frame
- removed link xtion_optical_frame
- removed link xtion_orbbec_aux_joint_frame
- removed link xtion_rgb_frame
- removed link xtion_rgb_optical_frame
- link xtion_link: geometry collision box size=0.04 0.185 0.03; visual mesh filename=tiago_description/meshes/sensors/xtion_pro_live/xtion_pro_l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
Joints:
- removed joint base_footprint_joint
- removed joint base_mic_back_left_joint
- removed joint base_mic_back_right_joint
- removed joint base_mic_front_left_joint
- removed joint base_mic_front_right_joint
- removed joint base_sonar_01_joint
- removed joint base_sonar_02_joint
- removed joint base_sonar_03_joint
- removed joint caster_back_left_1_joint
- removed joint caster_back_left_2_joint
- removed joint caster_back_right_1_joint
- removed joint caster_back_right_2_joint
- removed joint caster_front_left_1_joint
- removed joint caster_front_left_2_joint
- removed joint caster_front_right_1_joint
- removed joint caster_front_right_2_joint
- removed joint rgbd_laser_joint
- removed joint xtion_depth_joint
- removed joint xtion_depth_optical_joint
- removed joint xtion_optical_joint
- removed joint xtion_orbbec_aux_joint
- removed joint xtion_rgb_joint
- removed joint xtion_rgb_optical_joint
- joint cover_joint: origin xyz=0 0 0.13 rpy=0 0 0 -> xyz=0 0 0.0315 rpy=0 0 0; parent base_footprint -> base_link
- joint wheel_left_joint: limit effort=6.0 velocity=10.152284264 -> effort=10000.0 velocity=10000
- joint wheel_right_joint: limit effort=6.0 velocity=10.152284264 -> effort=1000.0 velocity=10000

Commit message: Cleans tiago urdf and removes unnessesary meshes. Adds structure to tiago env and adds tor-environment

File: tiagoReacher/resources/tiago_dual.urdf (robot description, URDF)
Before this commit: robot tiago_dual, 46 links, 45 joints
Links:
- added link caster_back_left_1_link, mass 0.05144761; visual mesh filename=pmb2_description/meshes/wheels/caster_1.stl
- added link caster_back_left_2_link, mass 0.08855784; collision cylinder length=0.001 radius=0.025; visual mesh filename=pmb2_description/meshes/wheels/caster_2.stl
- added link caster_back_right_1_link, mass 0.05144761; visual mesh filename=pmb2_description/meshes/wheels/caster_1.stl
- added link caster_back_right_2_link, mass 0.08855784; collision cylinder length=0.001 radius=0.025; visual mesh filename=pmb2_description/meshes/wheels/caster_2.stl
- added link caster_front_left_1_link, mass 0.05144761; visual mesh filename=pmb2_description/meshes/wheels/caster_1.stl
- added link caster_front_left_2_link, mass 0.08855784; collision cylinder length=0.001 radius=0.025; visual mesh filename=pmb2_description/meshes/wheels/caster_2.stl
- added link caster_front_right_1_link, mass 0.05144761; visual mesh filename=pmb2_description/meshes/wheels/caster_1.stl
- added link caster_front_right_2_link, mass 0.08855784; collision cylinder length=0.001 radius=0.025; visual mesh filename=pmb2_description/meshes/wheels/caster_2.stl
- link arm_left_5_link: geometry collision mesh filename=tiago_description/meshes/arm/arm_5_collision-wrist-2010.dae scale=-1 -1 -1; visual mesh filename=tiago_description/meshes/arm/arm_5-wrist-2010.stl scale=1 1 1
- link wheel_left_link: mass 1.82362 -> 100; geometry collision cylinder length=0.05 radius=0.1; visual mesh filename=pmb2_description/meshes/wheels/wheel.stl
- link wheel_right_link: mass 1.82362 -> 100; geometry collision cylinder length=0.05 radius=0.1; visual mesh filename=pmb2_description/meshes/wheels/wheel.stl
Joints:
- added joint caster_back_left_1_joint: type fixed, parent base_link, child caster_back_left_1_link, origin xyz=-0.1735 0.102 -0.0335 rpy=0 0 0, axis 0 0 1
- added joint caster_back_left_2_joint: type continuous, parent caster_back_left_1_link, child caster_back_left_2_link, origin xyz=-0.016 0.0000 -0.040 rpy=-1.57079632679 0 0, axis 0 0 1
- added joint caster_back_right_1_joint: type fixed, parent base_link, child caster_back_right_1_link, origin xyz=-0.1735 -0.102 -0.0335 rpy=0 0 0, axis 0 0 1
- added joint caster_back_right_2_joint: type continuous, parent caster_back_right_1_link, child caster_back_right_2_link, origin xyz=-0.016 0.0000 -0.040 rpy=-1.57079632679 0 0, axis 0 0 1
- added joint caster_front_left_1_joint: type fixed, parent base_link, child caster_front_left_1_link, origin xyz=0.1695 0.102 -0.0335 rpy=0 0 0, axis 0 0 1
- added joint caster_front_left_2_joint: type continuous, parent caster_front_left_1_link, child caster_front_left_2_link, origin xyz=-0.016 0.0000 -0.040 rpy=-1.57079632679 0 0, axis 0 0 1
- added joint caster_front_right_1_joint: type fixed, parent base_link, child caster_front_right_1_link, origin xyz=0.1695 -0.102 -0.0335 rpy=0 0 0, axis 0 0 1
- added joint caster_front_right_2_joint: type continuous, parent caster_front_right_1_link, child caster_front_right_2_link, origin xyz=-0.016 0.0000 -0.040 rpy=-1.57079632679 0 0, axis 0 0 1

Commit message: Adapts tiago to the the differential drive class.

File: tiagoReacher/resources/tiago_dual.urdf (robot description, URDF)
Before this commit: robot tiago_dual, 54 links, 53 joints
Joints:
- joint torso_lift_joint: limit lower=0 upper=0.35 effort=2000 velocity=0.07 -> lower=0 upper=0.35 effort=2000 velocity=0.35
