Commit message: Adds generic pointRobotUrdf environment as template for changes envised in other environments

File: pointRobotUrdf/resources/pointRobot.urdf (robot description, URDF)
Before this commit: robot pointRobot, 4 links, 3 joints
Links:
- added link lidar_link, mass 100.0; collision cylinder length=0.1 radius=0.02; visual cylinder length=0.1 radius=0.02
- added link lidar_sensor_link
- link base_link: geometry collision cylinder length=0.1 radius=0.2; visual cylinder length=0.1 radius=0.2
Joints:
- added joint lidar_sensor_joint: type fixed, parent lidar_link, child lidar_sensor_link, origin xyz=0 0 0.1 rpy=0 0 0
- added joint robot_lidar: type fixed, parent base_link, child lidar_link, origin xyz=0 0 0.1 rpy=0 0 0
- joint mobile_joint_theta: axis 0 0 1 -> (none); limit lower=-5 upper=5 effort=87 velocity=2.1750 -> (none); type revolute -> fixed
- joint mobile_joint_x: origin xyz=0 0 0.15 rpy=0 0 0 -> xyz=0 0 0.05 rpy=0 0 0

Commit message: Initializes multi-threading.

File: pointRobotUrdf/resources/pointRobot.urdf (robot description, URDF)
Before this commit: robot pointRobot, 6 links, 5 joints
Links:
- link lidar_sensor_link: mass None -> 1.0
