Commit message: Adds orientation correction for boxer.

File: urdfenvs/boxerRobot/resources/boxer.urdf (robot description, URDF)
Before this commit: robot albert, 7 links, 6 joints
Links:
- added link base_link_ori, mass 0.001
Joints:
- added joint base_add_orientation: type fixed, parent base_link_ori, child base_link, origin xyz=0.0 0 0 rpy=0 0 1.57079
