Commit message: Adds red dot on point robot and adds rotational degree of freedom.

File: urdfenvs/pointRobotUrdf/resources/pointRobot.urdf (robot description, URDF)
Before this commit: robot pointRobot, 6 links, 5 joints
Links:
- added link feature_link, mass 1.0; collision cylinder length=0.001 radius=0.02; visual cylinder length=0.001 radius=0.02
Joints:
- added joint feature_link_joint: type fixed, parent base_link, child feature_link, origin xyz=0 0.1 0.0505 rpy=0 0 0
- joint mobile_joint_theta: axis (none) -> 0 0 1; limit (none) -> lower=-5 upper=5 effort=87 velocity=2.1750; type fixed -> revolute
