Commit message: Adds visual links for sensor.

File: urdfenvs/braitenberg_robot/resources/braitenberg.urdf (robot description, URDF)
Before this commit: robot albert, 8 links, 7 joints
Links:
- removed link ee_link
- added link light_sensor_1_link; visual box size=0.1 0.01 0.1
- added link light_sensor_2_link; visual box size=0.1 0.01 0.1
Joints:
- removed joint ee_joint
- added joint light_sensor_1_joint: type fixed, parent base_link, child light_sensor_1_link, origin xyz=0.15 -0.37 0.07 rpy=0 0 0
- added joint light_sensor_2_joint: type fixed, parent base_link, child light_sensor_2_link, origin xyz=-0.15 -0.37 0.07 rpy=0 0 0

Commit message: change maximum speed of braitenberg vehicle

File: urdfenvs/braitenberg_robot/resources/braitenberg.urdf (robot description, URDF)
Before this commit: robot albert, 9 links, 8 joints
Links:
- link light_sensor_1_link: mass None -> 0.01
- link light_sensor_2_link: mass None -> 0.01

Commit message: changing direction of lightsensors

File: urdfenvs/braitenberg_robot/resources/braitenberg.urdf (robot description, URDF)
Before this commit: robot albert, 9 links, 8 joints
Joints:
- joint light_sensor_1_joint: origin xyz=0.15 -0.37 0.07 rpy=0 0 0 -> xyz=0.275 -0.25 0.07 rpy=0 0 4.7124
- joint light_sensor_2_joint: origin xyz=-0.15 -0.37 0.07 rpy=0 0 0 -> xyz=-0.275 -0.25 0.07 rpy=0 0 1.5708

Commit message: sensor-orientation

File: urdfenvs/braitenberg_robot/resources/braitenberg.urdf (robot description, URDF)
Before this commit: robot albert, 9 links, 8 joints
Joints:
- joint light_sensor_1_joint: origin xyz=0.275 -0.25 0.07 rpy=0 0 4.7124 -> xyz=0.275 -0.25 0.07 rpy=0 0 1.57079
- joint light_sensor_2_joint: origin xyz=-0.275 -0.25 0.07 rpy=0 0 1.5708 -> xyz=-0.275 -0.25 0.07 rpy=0 0 4.71239
