Commit message: 🚧 add quadrotor class, refine iris model

File: urdfenvs/iris/resources/iris.urdf (robot description, URDF)
Before this commit: robot iris, 6 links, 5 joints
Links:
- link iris__base_link: geometry collision box size=0.47 0.47 0.11; visual mesh filename=meshes/iris.stl scale=1 1 1
- link iris__rotor_0: geometry collision cylinder length=0.005 radius=0.128; visual mesh filename=meshes/iris_prop_ccw.dae scale=1 1 1
- link iris__rotor_1: geometry collision cylinder length=0.005 radius=0.128; visual mesh filename=meshes/iris_prop_ccw.dae scale=1 1 1
- link iris__rotor_2: geometry collision cylinder length=0.005 radius=0.128; visual mesh filename=meshes/iris_prop_cw.dae scale=1 1 1
- link iris__rotor_3: geometry collision cylinder length=0.005 radius=0.128; visual mesh filename=meshes/iris_prop_cw.dae scale=1 1 1
