Commit message: Adds end-effector to jackal robot.

File: urdfenvs/robots/jackal/jackal.urdf (robot description, URDF)
Before this commit: robot jackal, 13 links, 12 joints
Links:
- added link ee_link; visual sphere radius=0.05
Joints:
- added joint ee_joint: type fixed, parent base_link, child ee_link, origin xyz=0.2 0 0 rpy=0 0 0

Commit message: Cleans up mounting positions and mounting orientation. Fixes drone.

File: urdfenvs/robots/jackal/jackal.urdf (robot description, URDF)
Before this commit: robot jackal, 14 links, 13 joints
Links:
- link front_left_wheel_link: mass 0.000477 -> 1.0
- link front_right_wheel_link: mass 0.000477 -> 1.0

Commit message: Changes the lateral friction of castor wheels for differential drive robots to 0.

File: urdfenvs/robots/jackal/jackal.urdf (robot description, URDF)
Before this commit: robot jackal, 14 links, 13 joints
Links:
- link chassis_link: mass 10006.523 -> 6.523
- link rear_left_wheel_link: mass 100.477 -> 0.477
- link rear_right_wheel_link: mass 100.477 -> 0.477

Commit message: Corrects jackal to have two drivable axes. This is now an option for differential drive robots.

File: urdfenvs/robots/jackal/jackal.urdf (robot description, URDF)
Before this commit: robot jackal, 14 links, 13 joints
Joints:
- removed joint front_left_wheel_castor
- removed joint front_right_wheel_castor
- added joint front_left_wheel: type continuous, parent chassis_link, child front_left_wheel_link, origin xyz=0.131 0.187795 0.0345 rpy=0 0 0, axis 0 1 0, limit effort=10000 velocity=1000
- added joint front_right_wheel: type continuous, parent chassis_link, child front_right_wheel_link, origin xyz=0.131 -0.187795 0.0345 rpy=0 0 0, axis 0 1 0, limit effort=10000 velocity=1000
