Commit message: Adds heijn robot in examples.

File: examples/heijn_robot.urdf (robot description, URDF)
Before this commit: robot pointRobot, 7 links, 6 joints
Links:
- removed link lidar_link
- added link platform_link, mass 100.0; collision cylinder length=0.05 radius=0.05; visual cylinder length=0.05 radius=0.05
- added link pole_link, mass 100.0; collision cylinder length=0.43 radius=0.02; visual cylinder length=0.43 radius=0.02
- link base_link: geometry collision box size=0.61 0.33 0.13; visual box size=0.61 0.33 0.13
Joints:
- removed joint robot_lidar
- added joint platform_joint: type fixed, parent pole_link, child platform_link, origin xyz=0 0 0.2 rpy=0 0 0
- added joint robot_pole_joint: type fixed, parent base_link, child pole_link, origin xyz=0 0 0.1 rpy=0 0 0
- joint lidar_sensor_joint: parent lidar_link -> platform_link

Commit message: Adds collision links to heijn robot.

File: examples/heijn_robot.urdf (robot description, URDF)
Before this commit: robot pointRobot, 8 links, 7 joints
Links:
- added link collision_link_center_left, mass 0.01; visual sphere radius=0.12
- added link collision_link_center_right, mass 0.01; visual sphere radius=0.12
- added link collision_link_front_left, mass 0.01; visual sphere radius=0.12
- added link collision_link_front_right, mass 0.01; visual sphere radius=0.12
- added link collision_link_rear_left, mass 0.01; visual sphere radius=0.12
- added link collision_link_rear_right, mass 0.01; visual sphere radius=0.12
- link lidar_sensor_link: mass None -> 0.01
Joints:
- added joint collision_center_left_joint: type fixed, parent base_link, child collision_link_center_left, origin xyz=0.0 -0.13 0.0 rpy=0 0 0
- added joint collision_center_right_joint: type fixed, parent base_link, child collision_link_center_right, origin xyz=0.0 0.13 0.0 rpy=0 0 0
- added joint collision_front_left_joint: type fixed, parent base_link, child collision_link_front_left, origin xyz=0.22 -0.13 0.0 rpy=0 0 0
- added joint collision_front_right_joint: type fixed, parent base_link, child collision_link_front_right, origin xyz=0.22 0.13 0.0 rpy=0 0 0
- added joint collision_rear_left_joint: type fixed, parent base_link, child collision_link_rear_left, origin xyz=-0.22 -0.13 0.0 rpy=0 0 0
- added joint collision_rear_right_joint: type fixed, parent base_link, child collision_link_rear_right, origin xyz=-0.22 0.13 0.0 rpy=0 0 0

Commit message: Changes feature to front link.

File: examples/heijn_robot.urdf (robot description, URDF)
Before this commit: robot pointRobot, 14 links, 13 joints
Links:
- removed link feature_link
- added link front_link, mass 0.01; visual sphere radius=0.02
Joints:
- joint feature_link_joint: child feature_link -> front_link; origin xyz=0 0.1 0.0505 rpy=0 0 0 -> xyz=0.31 0.0 0.05 rpy=0 0 0

Commit message: Increases the size of the center collision obstacles.

File: examples/heijn_robot.urdf (robot description, URDF)
Before this commit: robot pointRobot, 14 links, 13 joints
Links:
- link collision_link_center_left: geometry visual sphere radius=0.20
- link collision_link_center_right: geometry visual sphere radius=0.20
Joints:
- removed joint feature_link_joint
- added joint front_link_joint: type fixed, parent base_link, child front_link, origin xyz=0.31 0.0 0.05 rpy=0 0 0
