Commit message: feat[sensors]: Moves lidar visualization to LidarSensor class.
Also fixes the other sensor with regards to inputs to the sense
function. Aligns the naming of the individual sensors.
Corrects test of obstacle sensing.

File: examples/pointRobot.urdf (robot description, URDF)
Before this commit: robot pointRobot, 7 links, 6 joints
Joints:
- joint lidar_sensor_joint: origin xyz=0 0 0.1 rpy=0 0 0 -> xyz=0 0 0.0 rpy=0 0 0
