Commit message: fix: Removes artificial rotation of boxer and albert.

File: urdfenvs/assets/albert/albert.urdf (robot description, URDF)
Before this commit: robot albert, 27 links, 26 joints
Links:
- removed link base_link_ori
Joints:
- removed joint base_add_orientation

File: urdfenvs/assets/boxer/boxer.urdf (robot description, URDF)
Before this commit: robot albert, 8 links, 7 joints
Links:
- removed link base_link_ori
Joints:
- removed joint base_add_orientation
